Commit message: 修正了orochi7_all.xacro文件中的基坐标

File: orochi_7dof_ws/src/orochi7/urdf/orochi7_all.xacro (robot description, xacro)
@@ -13,6 +13,12 @@
   </material>
 <!-- ##########################base_link########################## -->
-  <link name="dummy">
-    </link>
+  <!-- <link name="dummy">
+    </link> -->
+  <link name="world"/>
+  <joint name="virtual_joint" type="fixed">
+    <parent link="world"/>
+    <child link="base_link"/>
+    <origin rpy="0 0 0" xyz="0 0 0"/>
+  </joint>
   <link
     name="base_link">
@@ -55,9 +61,9 @@
     </collision>
   </link>
-  <joint name="dummy_joint" type="fixed">
+  <!-- <joint name="dummy_joint" type="fixed">
     <parent link="dummy"/>
     <child link="base_link"/>
     <origin xyz="0.0 0.0 0.2" rpy="0.0 0.0 0.0" />
-  </joint>
+  </joint> -->
 <!-- ##########################link_0########################## -->
   <link
